File: CM5-NAS.kicad_pcb (KiCad board)
At the start: 0 parts

Commit message: Started the power part of the schematic
looks very bad right now, but it's a work of art, trust me
Parts:
- added Module1: ComputeModule5-CM5, CM5:Raspberry-Pi-5-Compute-Module, F.Cu at (124.5, 109.5)
Other:
- board outline added: 40 x 55 mm
- copper layers 0 -> 2
