File: CM5-NAS.kicad_sch (KiCad schematic)
At the start: 0 parts

Commit message: Started the power part of the schematic
looks very bad right now, but it's a work of art, trust me
Parts:
- added Module1: ComputeModule5-CM5, CM5:Raspberry-Pi-5-Compute-Module, symbol CM5:ComputeModule5-CM5
Connections:
- new net GND: Module1.1 (GND), Module1.107 (GND), Module1.108 (GND), Module1.113 (GND), Module1.114 (GND), Module1.119 (GND), Module1.120 (GND), Module1.125 (GND), Module1.126 (GND), Module1.13 (GND), Module1.131 (GND), Module1.132 (GND)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
Other:
- added sheet Power (power.kicad_sch)
